File: main.kicad_sch (KiCad schematic)
At the start: 24 parts, among them J1 SERVEN, J2 JTAG, J3 SELECT, SW1 RESET, SW2 SERVEN, Y1 16MHz, Y2 32.768kHz

Commit message: Add AGND capacitors
Changed lines of the file:
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@@
-					(size 1.27 1.27)
-				)
-			)
-		)
-		(property "Value" "TPS3823-33"
-			(at 245.11 46.99 0)
-			(effects
-				(font
 					(size 1.27 1.27)
 				)
@@
 			)
 		)
+		(property "Value" "TPS3823-33"
+			(at 245.364 48.006 0)
+			(effects
+				(font
+					(size 1.27 1.27)
+				)
+			)
+		)

Commit message: Питание 5V от JTAG, множественные исправления
Parts:
- added D2: BAT60A, Diode_SMD:D_SOD-323, symbol Diode:BAT60A
Connections:
- net at J2.19 (DBGACK/NC): now also D2.2 (A)
- new net JTAGP: D2.1 (K)
- no-connect marks 0 -> 4
Other:
- moved on the sheet: J2, R4, R5, R7, R8, R9

Commit message: Обновление платы
Changed lines of the file:
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@@
 		(dnp no)
 		(property "Reference" "К1921ВГ015-1"
-			(at 126.238 41.91 0)
+			(at 123.952 41.91 0)
 			(effects
 				(font
@@
 			)
 		)
-		(property "Datasheet" "https://niiet.ru/wp-content/uploads/2025/02/%D0%A0%D0%9F-%D0%9A1921%D0%92%D0%93015_250219.pdf"
+		(property "Datasheet" "https://gitflic.ru/project/niiet/niiet_riscv_sdk/file?file=doc%2F%D0%9A1921VG015"
 			(at 135.636 99.568 90)
 			(effects
