File: К1921ВГ015.kicad_pcb (KiCad board)
At the start: 2 copper layers, 100 x 100 mm, 104 parts, among them J1 SERVEN, J11 Conn_02x05_Odd_Even, J12 AREF-TEST/MODULE, J14 Power DC 5V, J2 JTAG, J3 SELECT, J4 5V, J5 PORT-A-0-15, J6 Conn_02x22_Odd_Even, J7 Conn_02x22_Odd_Even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

Commit message: Питание 5V от JTAG, множественные исправления
Parts:
- added D2: BAT60A, Diode_SMD:D_SOD-323, B.Cu at (110.5, 100.0)
- J8: value Power Route -> Conn_02x04_Odd_Even; footprint Connector_PinHeader_2.54mm:PinHeader_2x03_P2.54mm_Vertical -> Connector_PinHeader_2.54mm:PinHeader_2x04_P2.54mm_Vertical
- moved D7 2.73 mm to (116.5, 51.5), turned to 180 degrees
- moved J8 2.51 mm to (119.5, 53.9)
- moved J11 0.40 mm to (119.5, 75.8)
Connections:
- J2 pad 19: unconnected-(J2-DBGACK/NC-Pad19) -> Net-(D2-A)
- U3 pad 5: unconnected-(U3-VCC-Pad5) -> 3.3L
- U8 pad 5: unconnected-(U8-VCC-Pad5) -> 3.3L
Routing:
- net PJTAG: track 0.00 -> 49.4 mm, vias 0 -> 2
- net Net-(J8-Pin_2): track 19.1 -> 29.4 mm
- net Net-(D2-A): track 0.00 -> 4.65 mm
- net 3.3L: track 51.3 -> 54.6 mm, vias 1 -> 3
- net MKUSBP: track 10.7 -> 8.38 mm
- net FTUSBP: track 45.9 -> 43.6 mm
- net Net-(D7-A): track 4.83 -> 2.70 mm
- net VCC1: track 469.8 -> 469.2 mm
- net GND1: vias 108 -> 109
Other:
- board text added: "DBG5V"

Commit message: Обновление платы
Parts:
- BT1: footprint Battery:Battery_Panasonic_CR2032-HFN_Horizontal_CircularHoles -> lib:BatteryHolder_CR1220_CR1225_SMT
- moved BT1 7.98 mm to (174.3, 57.8)
- moved C1 3.76 mm to (177.6, 70.7)
- moved C2 3.76 mm to (177.6, 68.2)
- moved R3 3.76 mm to (174.3, 69.4)
- moved Y1 3.76 mm to (170.9, 69.5)
- moved C8 1.48 mm to (171.2, 57.7)
- moved D1 1.43 mm to (174.3, 57.7)
- moved C9 1.40 mm to (177.4, 57.7)
Routing:
- net GNDL: track 75.5 -> 58.5 mm
- net VCC1: track 469.2 -> 454.7 mm
- net V_BAT: track 40.6 -> 36.8 mm
- net XI_OSC: track 31.8 -> 28.2 mm
- net XO_OSC: track 33.9 -> 30.5 mm
- net GND1: track 109.2 -> 106.0 mm, vias 109 -> 112
- net Net-(BT1-+): track 7.92 -> 7.33 mm, vias 0 -> 1
